File: Capacitijdmeter_ontwerp_officieel/Capacitijdmeter_ontwerp_officieel.kicad_sch (KiCad schematic)
At the start: 34 parts, among them J2 USB_C_Receptacle_PowerOnly_6P, SW2 SW_SPST, U0 74HC74, U1 74HC74, U10 4511, U12 7408, U14 74HC74, U15 74HC74, U16 4511, U2 7408, U20 74HC74, U21 74HC74, U22 4511, U27 74HC00, U28 74HC00, U29 74HC00, U3 4511, U4 74HC14, U7 74HC02, U8 74HC74, U9 74HC74

Commit message: add 4x3 switch
Parts:
- removed J2: USB_C_Receptacle_PowerOnly_6P, symbol Connector:USB_C_Receptacle_PowerOnly_6P
- added C10, C11, C12, C13, C14, C15, C16, C17, C18, C19, C20, C21, C5, C6, C7, C8, C9: 100nF, Capacitor_SMD:C_1206_3216Metric_Pad1.33x1.80mm_HandSolder, symbol Device:C
- added C22: C, symbol Device:C
- added R6: R, Resistor_SMD:R_1206_3216Metric_Pad1.30x1.75mm_HandSolder, symbol Device:R
- added R7: 8M1, Resistor_SMD:R_1206_3216Metric_Pad1.30x1.75mm_HandSolder, symbol Device:R
- added R8: 81k, Resistor_SMD:R_1206_3216Metric_Pad1.30x1.75mm_HandSolder, symbol Device:R
- added R9: 810R, Resistor_SMD:R_1206_3216Metric_Pad1.30x1.75mm_HandSolder, symbol Device:R
- added SW1: SW_Rotary_4x3, symbol Switch:SW_Rotary_4x3
- C1: value 150n -> scale-dependant C
- C3: footprint (none) -> Capacitor_SMD:C_1206_3216Metric_Pad1.33x1.80mm_HandSolder
- R1: value 10k -> scale-dependant R; footprint (none) -> Resistor_SMD:R_1206_3216Metric_Pad1.30x1.75mm_HandSolder
- R2: value Variable R -> scale-dependant R; footprint (none) -> Resistor_SMD:R_1206_3216Metric_Pad1.30x1.75mm_HandSolder
- R3, R5: value 5k1 -> R; footprint (none) -> Resistor_SMD:R_1206_3216Metric_Pad1.30x1.75mm_HandSolder
- R4: footprint (none) -> Resistor_SMD:R_1206_3216Metric_Pad1.30x1.75mm_HandSolder
- U10, U16, U22, U3: footprint Package_SO:SOIC-14_3.9x8.7mm_P1.27mm -> Package_SO:JEITA_SOIC-16_3.9x9.9mm_P1.27mm
- U11, U17, U23, U26: footprint (none) -> Display_7Segment:D1X8K
Connections:
- net +5V: now also C10.1, C11.1, C12.1, C13.1, C14.1, C15.1, C16.1, C17.2, C18.1, C19.1, C20.1, C21.1, C5.1, C6.1, C7.1, C8.1, C9.1; no longer C3.1, U2.14 (VCC), U2.14 (VCC), U2.14 (VCC)
- net GND: now also C10.2, C11.2, C12.2, C13.2, C14.2, C15.2, C16.2, C17.1, C18.2, C19.2, C20.2, C21.2, C22.2, C5.2, C6.2, C7.2, C8.2, C9.2, R7.2, R8.2, R9.2; no longer R2.2, R3.1, R5.1, U2.7 (GND), U2.7 (GND), U2.7 (GND)
- net V_{oscillator}: no longer U4.2
- net at C2.2, U28.4, U28.5: now also SW1.15; no longer R2.1
- net at R3.2: now also R5.2, U4.2, R6.2
- net at R4.2, SW2.1 (A), U27.2: no longer C4.1
- new net: R6.1, SW1.1
- new net: SW1.13, SW1.14, U4.1
- new net: R5.1, SW1.2
- new net: R3.1, SW1.3
- new net: C3.1, SW1.4
- new net: C4.1, SW1.5
- new net: C22.1, SW1.6
- new net: R7.1, SW1.7
- new net: R8.1, SW1.8
- new net: R9.1, SW1.9
- now unconnected: C1.1, R1.1
Other:
- moved on the sheet: C1, R1, U28E, U4A, U4G
