File: Capacitijdsmeter_ontwerp_meter/Capacitijdsmeter_ontwerp_meter/Capacitijdsmeter_ontwerp_meter.kicad_sch (KiCad schematic)
At the start: 22 parts, among them SW1 SW_Rotary_4x3, SW2 SW_SPST, U27 74HC00, U28 74HC00, U29 74HC00, U4 74HC14

Commit message: 17-10 meter + counter nieuwste
Parts:
- removed C1: scale-dependant C, symbol Device:C
- removed R2: scale-dependant R, Resistor_SMD:R_1206_3216Metric_Pad1.30x1.75mm_HandSolder, symbol Device:R
- added C16: 100pF, Capacitor_THT:C_Radial_D4.0mm_H5.0mm_P1.50mm, symbol Device:C
- added J1: DE9_Socket_MountingHoles, Connector_Dsub:DSUB-9_Socket_Horizontal_P2.77x2.84mm_EdgePinOffset7.70mm_Housed_MountingHolesOffset9.12mm, symbol Connector:DE9_Socket_MountingHoles
- added R10: 1M, Resistor_SMD:R_1206_3216Metric_Pad1.30x1.75mm_HandSolder, symbol Device:R
- added RV1: 1k, symbol Device:R_Potentiometer
- added RV2: 100k, symbol Device:R_Potentiometer
- added RV3: 5M, symbol Device:R_Potentiometer
- added unit 4 of U27
- added unit 2 of U4
- added unit 3 of U4
- C2: footprint (none) -> Connector_PinHeader_1.00mm:PinHeader_1x04_P1.00mm_Vertical
- R1: value scale-dependant R -> 460
- R7: value 8M1 -> 5M6
- R8: value 81k -> 30k
- R9: value 810R -> 300
- SW1: footprint (none) -> 43RotarySwitch1052Library:SW_CK1052
- renumbered U28 to U27, U29 to U27
Connections:
- net +5V: now also J1.6, J1.9
- net GND: now also R1.2, J1.1, J1.5, J1.7, J1.SH (PAD), RV1.2, RV2.2, RV3.2; no longer R7.2, R8.2, R9.2
- net V_{oneshot}: now also C16.1, U27.12
- net V_{oscillator}: now also R3.2, R5.2, R6.2, U4.2; no longer R1.2
- net at R1.1: now also C16.2, U4.3
- net at U27.10, U27.6, U27.9: no longer U27.1
- new net: U4.4, U4.5
- new net: U27.1, U27.11
- new net: R10.2, RV3.1
- new net: R8.2, RV2.1
- new net: R10.1, R7.2
- new net: R9.2, RV1.1
- new net V_{CounterMR}: J1.3
- new net V_{MR}: U4.6
- new net V_{Oneshot}: J1.4
- new net V_{Oscillator}: J1.8
- new net V_{Overflow}: J1.2, U27.13
Other:
- moved on the sheet: C14, C15, C22, C3, C4, R3, R5, R6, R7, R8, R9, SW1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

Commit message: pcb layout meter
Parts:
- added D1: LED, LED_THT:LED_D5.0mm, symbol Device:LED
- added J2: Barrel_Jack_Switch, Connector_BarrelJack:BarrelJack_Horizontal, symbol Connector:Barrel_Jack_Switch
- added R11: 345, Resistor_THT:R_Axial_DIN0207_L6.3mm_D2.5mm_P7.62mm_Horizontal, symbol Device:R
- C14, C15, C3: footprint Capacitor_SMD:C_1206_3216Metric_Pad1.33x1.80mm_HandSolder -> Capacitor_THT:C_Disc_D5.0mm_W2.5mm_P5.00mm
- C16: footprint Capacitor_THT:C_Radial_D4.0mm_H5.0mm_P1.50mm -> Capacitor_THT:C_Disc_D5.0mm_W2.5mm_P5.00mm
- C2: footprint Connector_PinHeader_1.00mm:PinHeader_1x04_P1.00mm_Vertical -> Capacitor_THT:C_Disc_D5.0mm_W2.5mm_P5.00mm
- C22, C4: footprint (none) -> Capacitor_THT:C_Disc_D5.0mm_W2.5mm_P5.00mm
- R1, R10, R3, R4, R5, R6, R7, R8, R9: footprint Resistor_SMD:R_1206_3216Metric_Pad1.30x1.75mm_HandSolder -> Resistor_THT:R_Axial_DIN0207_L6.3mm_D2.5mm_P7.62mm_Horizontal
- RV1, RV2, RV3: footprint (none) -> Potentiometer_THT:Potentiometer_ACP_CA14V-15_Vertical
- SW2: footprint (none) -> Button_Switch_THT:SW_Push_2P1T_Toggle_CK_PVA1xxH2xxxxxxV2
- U27, U4: footprint Package_SO:SOIC-14_3.9x8.7mm_P1.27mm -> Package_DIP:DIP-14_W7.62mm_Socket_LongPads
Connections:
- net V_{MR} is gone; now on net V_{CounterMR}: U4.6
- net V_{oneshot} is gone; now on net V_{Oneshot}: C16.1, U27.12, U27.8
- net V_{oscillator} is gone; now on net V_{Oscillator}: R3.2, R5.2, R6.2, U4.2
- net +5V: now also D1.2 (A), J2.1
- net GND: now also J2.2, R11.2
- new net: D1.1 (K), R11.1
Other:
- moved on the sheet: J1

Commit message: fix meter
Parts:
- removed unit 4 of U27
- added D2: LED, LED_THT:LED_D5.0mm, symbol Device:LED
- added R12: 345, Resistor_THT:R_Axial_DIN0207_L6.3mm_D2.5mm_P7.62mm_Horizontal, symbol Device:R
Connections:
- net V_{Overflow} is gone; now on net GND: J1.2
- net GND: now also R12.2
- net V_{Oneshot}: now also D2.2 (A)
- net at U27.1: now also U27.10, U27.6, U27.9
- new net: D2.1 (K), R12.1

Commit message: idk
Parts:
- added SW3: SW_SPST, Button_Switch_THT:SW_TH_Tactile_Omron_B3F-100x, symbol Switch:SW_SPST
- added unit 4 of U27
- added unit 6 of U4
- added unit 5 of U4
- added unit 4 of U4
- R1: value 460 -> 470
- RV1, RV2, RV3: footprint Potentiometer_THT:Potentiometer_ACP_CA14V-15_Vertical -> Potentiometer_THT:Potentiometer_Piher_PT-10-V10_Vertical
- SW2: footprint Button_Switch_THT:SW_Push_2P1T_Toggle_CK_PVA1xxH2xxxxxxV2 -> Button_Switch_THT:SW_SPST_Omron_B3F-40xx
Connections:
- net +5V: now also SW3.2 (B)
- net GND: now also U27.12, U27.13, U4.11, U4.13, U4.9
- net V_{CounterMR}: now also SW3.1 (A)

Commit message: "FUCKING HELL, IK WORD ZO BOOS BOOS :(((("
Parts:
- C22: value C -> 120n
- C3: value C -> 1n2
- C4: value C -> 12n
- R3, R5: value R -> 5k
- R6: value R -> 1k3
Connections:
- net V_{Oscillator}: no longer R3.2, R5.2
- net at SW1.1: no longer R6.1
- net at SW1.14, U4.1: now also R3.1; no longer SW1.13
- net at SW1.2: no longer R5.1
- net at SW1.3: no longer R3.1
- new net: R5.2, R6.1
- new net: R3.2, R5.1
