File: Capacitijdmeter_ontwerp_counter/Capacitijdmeter_ontwerp_counter.kicad_pcb (KiCad board)
At the start: 2 copper layers, 34 parts, among them U0 74HC74, U1 74HC74, U10 4511, U12 7408, U14 74HC74, U15 74HC74, U16 4511, U2 7408, U20 74HC74, U21 74HC74, U22 4511, U3 4511, U7 74HC02, U8 74HC74, U9 74HC74

Commit message: "goeiemorgen Koen, ga opnieuw alle traces doen"
Parts:
- added J1: Screw_Terminal_01x02, TerminalBlock:TerminalBlock_MaiXu_MX126-5.0-02P_1x02_P5.00mm, F.Cu at (254.0, 83.9)
- added J2: Screw_Terminal_01x02, TerminalBlock:TerminalBlock_MaiXu_MX126-5.0-02P_1x02_P5.00mm, F.Cu at (254.0, 71.2)
- added TP9: TestPoint, Connector_PinHeader_1.00mm:PinHeader_1x01_P1.00mm_Vertical, F.Cu at (154.9, 68.6)
- moved U8 86.1 mm to (219.9, 67.3), turned to 180 degrees
- moved U10 85.4 mm to (220.9, 56.2)
- moved C7 85.3 mm to (218.4, 75.2), turned to -90 degrees
- moved U11 81.8 mm to (214.7, 46.0)
- moved U20 76.2 mm to (243.9, 67.3), turned to 180 degrees
- moved C11 74.1 mm to (241.3, 75.2), turned to -90 degrees
- moved U12 73.8 mm to (241.2, 82.6), turned to 180 degrees
- moved U22 72.6 mm to (243.2, 56.2)
- moved U7 71.6 mm to (218.5, 83.5), turned to 180 degrees
- moved C19 71.3 mm to (214.5, 51.0), turned to 180 degrees
- moved U23 68.3 mm to (235.9, 46.0)
- moved C13 66.7 mm to (213.0, 88.9), turned to -90 degrees
- moved U9 65.8 mm to (207.9, 67.3), turned to 180 degrees
- moved C8 63.8 mm to (205.7, 75.2), turned to -90 degrees
- moved C17 59.3 mm to (236.0, 89.0)
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Connections:
- net Net-(U0A-Q) renamed Q_{FF12}
- net Net-(U0A-~{R}) renamed reset_3
- net Net-(U0B-Q) renamed Q_{FF13}
- net Net-(U10-DA) renamed Q_{FF4}
- net Net-(U10-DC) renamed Q_{FF6}
- net Net-(U10-Qa) renamed V_{a1}
- net Net-(U10-Qb) renamed V_{b1}
- net Net-(U10-Qc) renamed V_{c1}
- net Net-(U10-Qd) renamed V_{d1}
- net Net-(U10-Qe) renamed V_{e1}
- net Net-(U10-Qf) renamed V_{f1}
- net Net-(U10-Qg) renamed V_{g1}
- net Net-(U14A-Q) renamed Q_{FF8}
- net Net-(U14A-~{R}) renamed reset_2
- net Net-(U15A-Q) renamed Q_{FF10}
- net Net-(U16-Qa) renamed V_{a2}
- net Net-(U16-Qb) renamed V_{b2}
- net Net-(U16-Qc) renamed V_{c2}
- net Net-(U16-Qd) renamed V_{d2}
- net Net-(U16-Qe) renamed V_{e2}
- net Net-(U16-Qf) renamed V_{f2}
- net Net-(U16-Qg) renamed V_{g2}
- net Net-(U1A-Q) renamed Q_{FF14}
- net Net-(U1B-Q) renamed Q_{FF15}
- net Net-(U20A-C) renamed V_{input_counter}
- net Net-(U20A-Q) renamed Q_{FF0}
- net Net-(U20A-~{R}) renamed reset_0
- net Net-(U20B-Q) renamed Q_{FF1}
- net Net-(U21A-Q) renamed Q_{FF2}
- net Net-(U22-Qa) renamed V_{a0}
- net Net-(U22-Qb) renamed V_{b0}
- net Net-(U22-Qc) renamed V_{c0}
- net Net-(U22-Qd) renamed V_{d0}
- net Net-(U22-Qe) renamed V_{e0}
- net Net-(U22-Qf) renamed V_{f0}
- net Net-(U22-Qg) renamed V_{g0}
- net Net-(U8A-~{R}) renamed reset_1
- C16 pad 1: +5V -> GND
- C16 pad 2: GND -> +5V
- U0 pad 3: V_{clk0} -> V_{clk2}
- U10 pad 1: Net-(U10-DB) -> Q_{FF5}
- U10 pad 6: Net-(U10-DD) -> Q_{FF7}
- U14 pad 3: V_{clk2} -> V_{clk1}
- U14 pad 9: Net-(U14B-Q) -> Q_{FF9}
- U15 pad 9: Net-(U15B-Q) -> Q_{FF11}
- U16 pad 1: Net-(U14B-Q) -> Q_{FF9}
- U16 pad 6: Net-(U15B-Q) -> Q_{FF11}
- U2 pad 10: Net-(U15B-Q) -> Q_{FF7}
- U2 pad 11: V_{clk2} -> V_{clk0}
- U2 pad 13: Net-(U21B-Q) -> Q_{FF3}
- U2 pad 4: Net-(U10-DB) -> Q_{FF9}
- U2 pad 5: Net-(U10-DD) -> Q_{FF11}
- U2 pad 6: V_{clk0} -> V_{clk1}
- U2 pad 8: V_{clk1} -> V_{clk2}
- U2 pad 9: Net-(U14B-Q) -> Q_{FF5}
- U21 pad 11: Net-(U21A-D) -> unconnected-(U21B-C-Pad11)
- U21 pad 12: Net-(U21B-D) -> Q_{FF3}
- U21 pad 8: Net-(U21B-D) -> unconnected-(U21B-~{Q}-Pad8)
- U21 pad 9: Net-(U21B-Q) -> unconnected-(U21B-Q-Pad9)
- U22 pad 6: Net-(U21B-Q) -> Q_{FF3}
- U7 pad 12: V_{clk2} -> V_{clk0}
- U7 pad 6: V_{clk0} -> V_{clk1}
- U7 pad 9: V_{clk1} -> V_{clk2}
- U8 pad 3: V_{clk1} -> V_{clk0}
- U8 pad 9: Net-(U10-DB) -> Q_{FF5}
- U9 pad 9: Net-(U10-DD) -> Q_{FF7}
Routing:
- net Q_{FF3}: track 0.00 -> 120.1 mm
- net +5V: track 58.3 -> 169.9 mm, vias 0 -> 32
- net Q_{FF1}: track 0.00 -> 96.2 mm, vias 0 -> 2
- net Q_{FF7}: track 0.00 -> 73.8 mm
- net reset_3: track 17.2 -> 88.8 mm
- net V_{clk2}: track 0.00 -> 67.5 mm, vias 0 -> 2
- net V_{clk1}: track 0.00 -> 61.8 mm, vias 0 -> 3
- net V_{counteroverflow}: track 0.00 -> 60.0 mm, vias 0 -> 2
- net Q_{FF5}: track 0.00 -> 58.0 mm, vias 0 -> 2
- net Q_{FF11}: track 0.00 -> 48.4 mm, vias 0 -> 2
- net reset_2: track 0.00 -> 40.8 mm, vias 0 -> 2
- net reset_0: track 0.00 -> 40.3 mm, vias 0 -> 2
- net Q_{FF9}: track 0.00 -> 37.4 mm, vias 0 -> 2
- net Q_{FF15}: track 19.0 -> 52.5 mm, vias 0 -> 2
- net reset_1: track 0.00 -> 32.3 mm
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
Commit message: "PCB Fucking ontwerp"
Parts:
- removed J1, J2: Screw_Terminal_01x02, TerminalBlock:TerminalBlock_MaiXu_MX126-5.0-02P_1x02_P5.00mm
- added J3: DE9_Pins_MountingHoles, Connector_Dsub:DSUB-9_Pins_Horizontal_P2.77x2.84mm_EdgePinOffset7.70mm_Housed_MountingHolesOffset9.12mm, B.Cu at (146.0, 67.0)
- added R1: 10k, Resistor_THT:R_Axial_DIN0207_L6.3mm_D2.5mm_P10.16mm_Horizontal, F.Cu at (109.9, 25.0)
- added R2: 10k, Resistor_THT:R_Axial_DIN0207_L6.3mm_D2.5mm_P10.16mm_Horizontal, F.Cu at (131.1, 25.5)
- added R3: 10k, Resistor_THT:R_Axial_DIN0207_L6.3mm_D2.5mm_P10.16mm_Horizontal, F.Cu at (88.4, 25.5)
- added R4: 10k, Resistor_THT:R_Axial_DIN0207_L6.3mm_D2.5mm_P10.16mm_Horizontal, F.Cu at (67.4, 25.0)
- added TP1: TestPoint, Connector_PinHeader_1.00mm:PinHeader_1x01_P1.00mm_Vertical, F.Cu at (98.0, 83.0)
- added TP10: TestPoint, Connector_PinHeader_1.00mm:PinHeader_1x01_P1.00mm_Vertical, F.Cu at (118.5, 84.5)
- added TP11: TestPoint, Connector_PinHeader_1.00mm:PinHeader_1x01_P1.00mm_Vertical, F.Cu at (155.0, 52.0)
- added TP2: TestPoint, Connector_PinHeader_1.00mm:PinHeader_1x01_P1.00mm_Vertical, F.Cu at (91.5, 64.0)
- added TP3: TestPoint, Connector_PinHeader_1.00mm:PinHeader_1x01_P1.00mm_Vertical, F.Cu at (70.0, 60.5)
- added TP5: TestPoint, Connector_PinHeader_1.00mm:PinHeader_1x01_P1.00mm_Vertical, F.Cu at (132.0, 89.5)
- added TP6: TestPoint, Connector_PinHeader_1.00mm:PinHeader_1x01_P1.00mm_Vertical, F.Cu at (139.5, 86.5)
- added TP7: TestPoint, Connector_PinHeader_1.00mm:PinHeader_1x01_P1.00mm_Vertical, F.Cu at (139.0, 81.0)
- added TP8: TestPoint, Connector_PinHeader_1.00mm:PinHeader_1x01_P1.00mm_Vertical, F.Cu at (142.0, 58.5)
- U11, U17, U23, U26: footprint Display_7Segment:D1X8K -> footprints:SC56-11EWA_KNB
- moved TP9 112.2 mm to (43.0, 76.5)
- moved C20 110.5 mm to (81.5, 50.4)
- moved C21 110.5 mm to (126.5, 50.5)
- moved U12 110.1 mm to (131.1, 82.0)
- moved U22 110.1 mm to (133.1, 55.6)
- moved U0 110.1 mm to (61.7, 66.7), turned to -90 degrees
- moved U10 110.1 mm to (110.8, 55.6)
- moved U11 110.1 mm to (104.6, 45.4)
- moved U15 110.1 mm to (73.7, 66.7), turned to -90 degrees
- moved U16 110.1 mm to (88.5, 55.6)
- moved U17 110.1 mm to (83.4, 45.4)
- moved U21 110.1 mm to (121.8, 66.7), turned to -90 degrees
- moved U3 110.1 mm to (66.2, 55.6)
- moved U7 110.1 mm to (108.3, 82.9)
- moved U8 110.1 mm to (109.7, 66.7), turned to -90 degrees
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Connections:
- net V_{counteroverflow} renamed V_{Counteroverflow}
- U11 pad 3: GND -> Net-(R1-Pad1)
- U11 pad 8: GND -> Net-(R1-Pad1)
- U17 pad 3: GND -> Net-(R3-Pad1)
- U17 pad 8: GND -> Net-(R3-Pad1)
- U21 pad 11: unconnected-(U21B-C-Pad11) -> Net-(U21A-D)
- U21 pad 12: Q_{FF3} -> Net-(U21B-D)
- U21 pad 8: unconnected-(U21B-~{Q}-Pad8) -> Net-(U21B-D)
- U21 pad 9: unconnected-(U21B-Q-Pad9) -> Q_{FF3}
- U23 pad 3: GND -> Net-(R2-Pad1)
- U23 pad 5: GND -> unconnected-(U23-DP-Pad5)
- U23 pad 8: GND -> Net-(R2-Pad1)
- U26 pad 3: GND -> Net-(R4-Pad1)
- U26 pad 8: GND -> Net-(R4-Pad1)
Routing:
- net +5V: track 169.9 -> 596.2 mm, vias 32 -> 34
- net V_{Counteroverflow}: track 60.0 -> 113.3 mm
- net V_{CounterMR}: track 17.5 -> 69.0 mm, vias 0 -> 1
- net reset_0: track 40.3 -> 72.9 mm, vias 2 -> 0
- net Q_{FF3}: track 120.1 -> 88.4 mm, vias 0 -> 2
- net V_{clk2}: track 67.5 -> 95.9 mm
- net Net-(R4-Pad1): track 0.00 -> 25.5 mm
- net V_{clk0}: track 70.9 -> 95.5 mm, vias 2 -> 3
- net V_{clk1}: track 61.8 -> 84.1 mm
- net Net-(R1-Pad1): track 0.00 -> 20.5 mm
- net Net-(R2-Pad1): track 0.00 -> 20.0 mm
- net Net-(R3-Pad1): track 0.00 -> 19.9 mm
- net V_{input_counter}: track 18.8 -> 32.2 mm, vias 0 -> 2
- net V_{f0}: track 29.8 -> 42.8 mm
- net Q_{FF1}: track 96.2 -> 83.4 mm
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- added copper zone on B.Cu, net GND
- added copper zone on F.Cu, net GND

Commit message: "alles behalve de ding geroute"
Parts:
- removed C16: 100nF, Capacitor_SMD:C_1206_3216Metric_Pad1.33x1.80mm_HandSolder
- removed the R2 at (131.1, 25.5)
- removed R4: 10k, Resistor_THT:R_Axial_DIN0207_L6.3mm_D2.5mm_P10.16mm_Horizontal
- removed TP9: TestPoint, Connector_PinHeader_1.00mm:PinHeader_1x01_P1.00mm_Vertical
- removed U0, U1: 74HC74, Package_SO:SOIC-14_3.9x8.7mm_P1.27mm
- removed U26: ~, footprints:SC56-11EWA_KNB
- removed U3: 4511, Package_SO:JEITA_SOIC-16_3.9x9.9mm_P1.27mm
- added R2: 10k, Resistor_SMD:R_1206_3216Metric_Pad1.30x1.75mm_HandSolder, B.Cu at (53.0, 25.8)
- added R2: 10k, Resistor_SMD:R_1206_3216Metric_Pad1.30x1.75mm_HandSolder, B.Cu at (77.0, 25.8)
- added U20: 74HC74, Package_SO:SOIC-14_3.9x8.7mm_P1.27mm, B.Cu at (110.9, 66.4)
- added U21: 74HC74, Package_SO:SOIC-14_3.9x8.7mm_P1.27mm, B.Cu at (122.9, 66.4)
- added U22: 4511, Package_SO:JEITA_SOIC-16_3.9x9.9mm_P1.27mm, B.Cu at (121.8, 55.2)
- added U23: ~, footprints:SC56-11EWA_KNB, F.Cu at (116.9, 45.1)
- C10, C11, C12, C13, C17, C18, C19, C20, C21, C5, C6, C7, C8, C9, U10, U12, U14, U15, U16, U2, U20, U21, U22, U7, U8, U9: moved to B.Cu
- R1, R3: footprint Resistor_THT:R_Axial_DIN0207_L6.3mm_D2.5mm_P10.16mm_Horizontal -> Resistor_SMD:R_1206_3216Metric_Pad1.30x1.75mm_HandSolder; moved to B.Cu
- moved TP8 103.9 mm to (38.1, 61.0)
- moved C11 102.7 mm to (35.8, 76.2)
- moved U20 93.2 mm to (40.6, 66.7)
- moved U12 87.9 mm to (43.2, 83.8), turned to 0 degrees
- moved U22 81.6 mm to (51.4, 55.6)
- moved U23 79.2 mm to (46.6, 45.4)
- moved C12 78.7 mm to (47.8, 76.2)
- moved C17 77.4 mm to (48.5, 88.4)
- moved C18 70.5 mm to (129.7, 53.0), turned to 0 degrees
- moved U21 69.2 mm to (52.6, 66.7)
- moved C21 67.2 mm to (59.4, 53.3), turned to 0 degrees
- moved C6 64.2 mm to (118.2, 75.9)
- moved C7 55.2 mm to (59.8, 76.2)
- moved U8 45.2 mm to (64.6, 66.7)
- moved U2 44.6 mm to (109.5, 82.9), turned to 180 degrees
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Routing:
- net +5V: track 596.2 -> 0.00 mm, vias 34 -> 0
- net V_{Counteroverflow}: track 113.3 -> 0.00 mm, vias 2 -> 0
- net V_{clk2}: track 95.9 -> 0.00 mm, vias 2 -> 0
- net V_{clk0}: track 95.5 -> 0.00 mm, vias 3 -> 0
- net reset_3: track 86.9 -> 0.00 mm, vias 2 -> 0
- net V_{clk1}: track 84.1 -> 0.00 mm, vias 3 -> 0
- net V_{CounterMR}: track 69.0 -> 0.00 mm, vias 1 -> 0
- net Q_{FF15}: track 57.3 -> 0.00 mm, vias 2 -> 0
- net Q_{FF7}: track 76.6 -> 22.5 mm
- net Net-(U20A-D): track 19.6 -> 72.5 mm, vias 1 -> 0
- net Q_{FF5}: track 65.5 -> 20.7 mm, vias 2 -> 0
- net Q_{FF3}: track 88.4 -> 45.0 mm, vias 2 -> 0
- net Q_{FF1}: track 83.4 -> 41.4 mm, vias 2 -> 0
- net V_{f3}: track 38.7 -> 0.00 mm, vias 1 -> 0
- net V_{f0}: track 42.8 -> 81.1 mm, vias 1 -> 0
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- removed copper zone on B.Cu, net GND
- removed copper zone on F.Cu, net GND

Commit message: "flipping hell, Koen, hier asjeblieft"
Parts:
- added C16: 100nF, Capacitor_SMD:C_1206_3216Metric_Pad1.33x1.80mm_HandSolder, B.Cu at (165.1, 97.7)
- added TP9: TestPoint, Connector_PinHeader_1.00mm:PinHeader_1x01_P1.00mm_Vertical, F.Cu at (58.4, 88.9)
- C10: renamed from C8; moved to F.Cu
- C12: renamed from C6; moved to F.Cu
- C6: renamed from C12; moved to F.Cu
- C8: renamed from C10; moved to F.Cu
- U2, U7: moved to F.Cu
- moved U12 78.4 mm to (121.6, 83.1), turned to 180 degrees
- moved U7 19.8 mm to (85.7, 85.0), turned to 90 degrees
- moved U2 11.8 mm to (97.7, 84.1), turned to -90 degrees
- renumbered C5 to C11, C21 to C18, C20 to C19, C19 to C20, C18 to C21, C11 to C5, C9 to C7, C7 to C9, R3 to R2, R2 to R3, R2 to R4, TP2 to TP1, TP1 to TP2, TP8 to TP3, TP3 to TP8, U20 to U0, U21 to U1, U16 to U10, U17 to U11, U8 to U14, U9 to U15, U10 to U16, U11 to U17, U23 to U26, U22 to U3, U14 to U8, U15 to U9
Connections:
- R2 pad 1: Net-(R3-Pad1) -> Net-(R2-Pad1)
- R3 pad 1: Net-(R2-Pad1) -> Net-(R3-Pad1)
- R4 pad 1: Net-(R2-Pad1) -> Net-(R4-Pad1)
- TP1 pad 1: V_{clk1} -> V_{clk0}
- TP2 pad 1: V_{clk0} -> V_{clk1}
- TP3 pad 1: Net-(U20A-D) -> V_{clk2}
- TP8 pad 1: V_{clk2} -> Net-(U20A-D)
- U0 pad 1: reset_0 -> reset_3
- U0 pad 11: Net-(U20A-D) -> Net-(U0A-D)
- U0 pad 12: Net-(U20B-D) -> Net-(U0B-D)
- U0 pad 13: reset_0 -> reset_3
- U0 pad 2: Net-(U20A-D) -> Net-(U0A-D)
- U0 pad 3: V_{input_counter} -> V_{clk2}
- U0 pad 5: Q_{FF0} -> Q_{FF12}
- U0 pad 6: Net-(U20A-D) -> Net-(U0A-D)
- U0 pad 8: Net-(U20B-D) -> Net-(U0B-D)
- U0 pad 9: Q_{FF1} -> Q_{FF13}
- U1 pad 1: reset_0 -> reset_3
- U1 pad 11: Net-(U21A-D) -> Net-(U1A-D)
- U1 pad 12: Net-(U21B-D) -> Net-(U1B-D)
- U1 pad 13: reset_0 -> reset_3
- U1 pad 2: Net-(U21A-D) -> Net-(U1A-D)
- U1 pad 3: Net-(U20B-D) -> Net-(U0B-D)
- U1 pad 5: Q_{FF2} -> Q_{FF14}
- U1 pad 6: Net-(U21A-D) -> Net-(U1A-D)
- U1 pad 8: Net-(U21B-D) -> Net-(U1B-D)
- U1 pad 9: Q_{FF3} -> Q_{FF15}
- U10 pad 1: Q_{FF9} -> Q_{FF5}
- U10 pad 10: V_{d2} -> V_{d1}
- U10 pad 11: V_{c2} -> V_{c1}
- U10 pad 12: V_{b2} -> V_{b1}
- U10 pad 13: V_{a2} -> V_{a1}
- U10 pad 14: V_{g2} -> V_{g1}
- U10 pad 15: V_{f2} -> V_{f1}
- U10 pad 2: Q_{FF10} -> Q_{FF6}
- U10 pad 6: Q_{FF11} -> Q_{FF7}
- U10 pad 7: Q_{FF8} -> Q_{FF4}
- U10 pad 9: V_{e2} -> V_{e1}
- U11 pad 1: V_{e2} -> V_{e1}
- U11 pad 10: V_{g2} -> V_{g1}
- U11 pad 2: V_{d2} -> V_{d1}
- U11 pad 3: Net-(R3-Pad1) -> Net-(R1-Pad1)
- U11 pad 4: V_{c2} -> V_{c1}
- U11 pad 6: V_{b2} -> V_{b1}
- U11 pad 7: V_{a2} -> V_{a1}
- U11 pad 8: Net-(R3-Pad1) -> Net-(R1-Pad1)
- U11 pad 9: V_{f2} -> V_{f1}
- U14 pad 1: reset_1 -> reset_2
- U14 pad 13: reset_1 -> reset_2
- U14 pad 3: V_{clk0} -> V_{clk1}
- U14 pad 5: Q_{FF4} -> Q_{FF8}
- U14 pad 9: Q_{FF5} -> Q_{FF9}
- U15 pad 1: reset_1 -> reset_2
- U15 pad 13: reset_1 -> reset_2
- U15 pad 5: Q_{FF6} -> Q_{FF10}
- U15 pad 9: Q_{FF7} -> Q_{FF11}
- U16 pad 1: Q_{FF5} -> Q_{FF9}
- U16 pad 10: V_{d1} -> V_{d2}
- U16 pad 11: V_{c1} -> V_{c2}
- U16 pad 12: V_{b1} -> V_{b2}
- U16 pad 13: V_{a1} -> V_{a2}
- U16 pad 14: V_{g1} -> V_{g2}
- U16 pad 15: V_{f1} -> V_{f2}
- U16 pad 2: Q_{FF6} -> Q_{FF10}
- U16 pad 6: Q_{FF7} -> Q_{FF11}
- U16 pad 7: Q_{FF4} -> Q_{FF8}
- U16 pad 9: V_{e1} -> V_{e2}
- U17 pad 1: V_{e1} -> V_{e2}
- U17 pad 10: V_{g1} -> V_{g2}
- U17 pad 2: V_{d1} -> V_{d2}
- U17 pad 3: Net-(R1-Pad1) -> Net-(R3-Pad1)
- U17 pad 4: V_{c1} -> V_{c2}
- U17 pad 6: V_{b1} -> V_{b2}
- U17 pad 7: V_{a1} -> V_{a2}
- U17 pad 8: Net-(R1-Pad1) -> Net-(R3-Pad1)
- U17 pad 9: V_{f1} -> V_{f2}
- U26 pad 1: V_{e0} -> V_{e3}
- U26 pad 10: V_{g0} -> V_{g3}
- U26 pad 2: V_{d0} -> V_{d3}
- U26 pad 3: Net-(R2-Pad1) -> Net-(R4-Pad1)
- U26 pad 4: V_{c0} -> V_{c3}
- U26 pad 5: unconnected-(U23-DP-Pad5) -> GND
- U26 pad 6: V_{b0} -> V_{b3}
- U26 pad 7: V_{a0} -> V_{a3}
- U26 pad 8: Net-(R2-Pad1) -> Net-(R4-Pad1)
- U26 pad 9: V_{f0} -> V_{f3}
- U3 pad 1: Q_{FF1} -> Q_{FF13}
- U3 pad 10: V_{d0} -> V_{d3}
- U3 pad 11: V_{c0} -> V_{c3}
- U3 pad 12: V_{b0} -> V_{b3}
- U3 pad 13: V_{a0} -> V_{a3}
- U3 pad 14: V_{g0} -> V_{g3}
- U3 pad 15: V_{f0} -> V_{f3}
- U3 pad 2: Q_{FF2} -> Q_{FF14}
- U3 pad 6: Q_{FF3} -> Q_{FF15}
- U3 pad 7: Q_{FF0} -> Q_{FF12}
- U3 pad 9: V_{e0} -> V_{e3}
- U8 pad 1: reset_2 -> reset_1
- U8 pad 13: reset_2 -> reset_1
- U8 pad 3: V_{clk1} -> V_{clk0}
- U8 pad 5: Q_{FF8} -> Q_{FF4}
- U8 pad 9: Q_{FF9} -> Q_{FF5}
- U9 pad 1: reset_2 -> reset_1
- U9 pad 13: reset_2 -> reset_1
- U9 pad 5: Q_{FF10} -> Q_{FF6}
- U9 pad 9: Q_{FF11} -> Q_{FF7}
Routing:
- net +5V: track 0.00 -> 233.7 mm, vias 0 -> 12
- net V_{f0}: track 81.1 -> 40.5 mm
- net V_{f3}: track 0.00 -> 40.5 mm
- net V_{g3}: track 0.00 -> 32.7 mm
- net V_{g0}: track 65.3 -> 32.7 mm
- net V_{a3}: track 0.00 -> 32.1 mm
- net V_{a0}: track 64.3 -> 32.1 mm
- net reset_3: track 0.00 -> 28.6 mm
- net reset_0: track 55.8 -> 28.6 mm
- net V_{b3}: track 0.00 -> 27.0 mm
- net V_{b0}: track 54.0 -> 27.0 mm
- net Net-(U0B-D): track 0.00 -> 23.9 mm
- net Q_{FF3}: track 45.0 -> 22.5 mm
- net Q_{FF15}: track 0.00 -> 22.5 mm
- net Q_{FF1}: track 41.4 -> 20.7 mm
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
Commit message: s
Parts:
- removed U12: 7408, Package_SO:SOIC-14_3.9x8.7mm_P1.27mm
- added C14: 100nF, Capacitor_SMD:C_1206_3216Metric_Pad1.33x1.80mm_HandSolder, F.Cu at (2.50, 1.18)
- added U4: 7402, Package_SO:SOIC-14_3.9x8.7mm_P1.27mm, B.Cu at (126.9, 83.8)
- added U5: 7411, Package_SO:SOIC-14_3.9x8.7mm_P1.27mm, F.Cu at (126.9, 83.8)
- moved U7 27.0 mm to (71.2, 62.2), turned to 0 degrees
- moved TP5 18.5 mm to (137.2, 96.5)
- moved TP6 17.8 mm to (142.2, 96.5)
- moved U2 16.3 mm to (88.0, 71.1), turned to 90 degrees
- moved TP10 15.4 mm to (101.6, 99.1)
- moved TP7 5.41 mm to (129.5, 76.2)
Connections:
- net reset_0 renamed Net-(U20A-~{R})
- net reset_1 renamed Net-(U8A-~{R})
- net reset_2 renamed Net-(U14A-~{R})
- J3 pad 2: V_{Counteroverflow} -> GND
Routing:
- net V_{CounterMR}: track 0.00 -> 16.6 mm
- net Net-(U4-Pad13): track 0.00 -> 7.32 mm
- net V_{Counterstop}: track 0.00 -> 1.27 mm

Commit message: dih
Parts:
- removed TP10: TestPoint, Connector_PinHeader_1.00mm:PinHeader_1x01_P1.00mm_Vertical
- C14: moved to B.Cu
- moved C14 153.5 mm to (127.0, 91.0)
- moved U7 24.6 mm to (95.5, 66.0), turned to 90 degrees
- moved U2 18.6 mm to (89.8, 52.5)
- moved U5 10.5 mm to (116.5, 83.8)
Routing:
- net Q_{FF13}: track 20.7 -> 66.7 mm, vias 0 -> 1
- net Q_{FF3}: track 22.5 -> 62.5 mm, vias 0 -> 1
- net Q_{FF1}: track 20.7 -> 57.8 mm, vias 0 -> 1
- net Q_{FF15}: track 22.5 -> 54.6 mm, vias 0 -> 1
- net V_{clk0}: track 0.00 -> 20.9 mm
- net Q_{FF5}: track 20.7 -> 39.1 mm, vias 0 -> 1
- net Net-(U20A-D): track 54.4 -> 36.4 mm
- net Q_{FF7}: track 22.5 -> 38.1 mm, vias 0 -> 1
- net Net-(U8A-D): track 0.00 -> 14.8 mm
- net Net-(U0A-D): track 0.00 -> 14.8 mm
- net +5V: track 233.7 -> 246.1 mm
- net V_{clk2}: track 18.1 -> 21.6 mm
- net V_{CounterMR}: track 16.6 -> 17.8 mm

Commit message: "FUCKING HELL, IK WORD ZO BOOS BOOS :(((("
Parts:
- moved J3 29.3 mm to (134.9, 37.6)
- moved C14 24.6 mm to (145.2, 74.5)
- moved TP7 24.6 mm to (147.8, 59.7)
- moved U5 22.7 mm to (132.0, 67.3)
- moved U4 22.5 mm to (142.2, 67.3)
- moved TP5 19.3 mm to (129.5, 78.7)
- moved TP6 19.3 mm to (134.6, 78.7)
- moved C16 19.3 mm to (157.4, 79.9)
- moved U7 14.0 mm to (83.8, 73.7)
- moved U2 13.2 mm to (82.5, 63.6)
- moved TP1 2.54 mm to (85.6, 58.4)
Routing:
- net Q_{FF15}: track 54.6 -> 25.6 mm
- net Q_{FF13}: track 66.7 -> 48.8 mm
- net V_{CounterMR}: track 17.8 -> 0.00 mm
- net V_{clk2}: track 21.6 -> 3.88 mm
- net V_{clk0}: track 20.9 -> 6.30 mm
- net V_{clk1}: track 0.00 -> 12.7 mm
- net Q_{FF1}: track 57.8 -> 66.3 mm
- net +5V: track 246.1 -> 238.3 mm
- net Net-(U4-Pad13): track 7.32 -> 0.00 mm
- net Q_{FF3}: track 62.5 -> 67.2 mm
- net Q_{FF5}: track 39.1 -> 42.3 mm
- net Q_{FF7}: track 38.1 -> 39.9 mm
- net V_{Counterstop}: track 1.27 -> 0.00 mm
- net Net-(U8B-D): track 23.9 -> 23.4 mm

Commit message: "NIEUWE VERSIE ERIN GEKNIKKERD MET EEN PCB DAT BIJNA KLAAR IS"
Parts:
- C13, C16: moved to F.Cu
- U5: moved to B.Cu
- moved C17 88.0 mm to (134.2, 68.7)
- moved C16 75.9 mm to (86.4, 53.3)
- moved TP5 28.4 mm to (134.6, 50.8)
- moved TP6 25.5 mm to (137.2, 53.3)
- moved TP7 24.6 mm to (129.5, 76.2)
- moved TP11 15.6 mm to (142.2, 61.0)
- moved TP9 13.0 mm to (55.9, 76.2)
- moved C14 8.96 mm to (142.2, 66.0), turned to 180 degrees
- moved U5 6.86 mm to (134.6, 61.0)
- moved C13 6.74 mm to (75.1, 82.7)
- moved U4 6.35 mm to (142.2, 73.7), turned to 180 degrees
- moved U2 6.19 mm to (79.1, 58.4), turned to 0 degrees
- moved J3 6.12 mm to (140.8, 36.0)
- moved C8 5.42 mm to (95.3, 81.6)
- moved C20 2.89 mm to (84.8, 50.8)
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Connections:
- J3 pad 1: unconnected-(J3-Pad1) -> GND
Routing:
- net +5V: track 238.3 -> 692.6 mm, vias 12 -> 27
- net V_{CounterMR}: track 0.00 -> 145.7 mm, vias 0 -> 3
- net V_{clk2}: track 3.88 -> 120.1 mm, vias 0 -> 1
- net V_{Counteroverflow}: track 0.00 -> 107.5 mm, vias 0 -> 3
- net reset_3: track 28.6 -> 95.4 mm, vias 0 -> 1
- net V_{input_counter}: track 0.00 -> 58.2 mm, vias 0 -> 2
- net V_{clk0}: track 6.30 -> 61.9 mm, vias 0 -> 3
- net Net-(U20A-~{R}): track 28.6 -> 66.0 mm, vias 0 -> 1
- net V_{oscillator}: track 0.00 -> 29.7 mm
- net V_{clk1}: track 12.7 -> 41.8 mm, vias 0 -> 1
- net V_{oneshot}: track 0.00 -> 23.7 mm
- net Net-(U20A-D): track 36.4 -> 18.2 mm
- net Q_{FF15}: track 25.6 -> 42.7 mm
- net V_{Counterstop}: track 0.00 -> 17.0 mm
- net Q_{FF9}: track 20.7 -> 36.2 mm, vias 0 -> 1
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