File: Capacitijdmeter_ontwerp_counter/Capacitijdmeter_ontwerp_counter.kicad_pcb (KiCad board)
At the start: 2 copper layers, 50 parts, among them J3 DE9_Pins_MountingHoles, U0 74HC74, U1 74HC74, U10 4511, U14 74HC74, U15 74HC74, U16 4511, U2 7408, U20 74HC74, U21 74HC74, U22 4511, U3 4511, U4 7402, U5 7411, U7 74HC02, U8 74HC74, U9 74HC74

Commit message: "ALL COMMIT"
Parts:
- C13: moved to B.Cu
- R1, R2, R3, R4: value 10k -> 500
- moved C13 10.4 mm to (84.2, 87.6), turned to 180 degrees
- moved C11 7.62 mm to (106.2, 83.5)
- moved C12 7.62 mm to (118.2, 83.5)
- moved U0 7.62 mm to (40.6, 74.3)
- moved U1 7.62 mm to (52.6, 74.3)
- moved U14 7.62 mm to (64.6, 74.3)
- moved U15 7.62 mm to (76.6, 74.3)
- moved U4 7.62 mm to (142.2, 81.3)
- moved U8 7.62 mm to (88.0, 74.3)
- moved U9 7.62 mm to (100.0, 74.3)
- moved U5 7.62 mm to (134.6, 68.6)
- moved C10 7.62 mm to (71.8, 86.1)
- moved C14 7.62 mm to (142.2, 73.7)
- moved C17 7.62 mm to (134.2, 76.3)
- moved C5 7.62 mm to (35.8, 83.8)
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Connections:
- U23 pad 5: unconnected-(U23-DP-Pad5) -> GND
Routing:
- net +5V: track 692.6 -> 870.4 mm, vias 27 -> 34
- net V_{Counteroverflow}: track 107.5 -> 130.4 mm
- net V_{clk1}: track 41.8 -> 60.9 mm
- net V_{clk0}: track 61.9 -> 78.1 mm, vias 3 -> 5
- net V_{input_counter}: track 58.2 -> 74.3 mm
- net Q_{FF7}: track 40.0 -> 55.8 mm
- net Q_{FF4}: track 15.8 -> 30.1 mm
- net Net-(U8A-~{R}): track 40.1 -> 53.4 mm, vias 0 -> 1
- net Q_{FF5}: track 36.8 -> 48.7 mm
- net Q_{FF15}: track 42.7 -> 53.4 mm
- net Q_{FF9}: track 36.2 -> 46.6 mm
- net Q_{FF8}: track 13.4 -> 23.7 mm
- net V_{CounterMR}: track 145.7 -> 155.8 mm
- net V_{clk2}: track 120.1 -> 129.8 mm
- net Q_{FF1}: track 62.2 -> 71.6 mm
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- added copper zone on B.Cu, net GND
- added copper zone on F.Cu, net GND
Other:
- board outline added: 118.5 x 80.8 mm

Commit message: "DRC verwijderen"
Parts:
- moved TP8 1.68 mm to (107.9, 62.2)
- moved TP1 0.11 mm to (86.3, 58.5)
Routing:
- net V_{CounterMR}: track 155.8 -> 161.7 mm
- net Net-(U20A-D): track 25.9 -> 20.8 mm
- net +5V: track 870.4 -> 874.8 mm, vias 34 -> 33
- net Q_{FF11}: track 41.8 -> 37.6 mm
- net Q_{FF9}: track 46.6 -> 50.5 mm
- net Q_{FF7}: track 55.8 -> 53.3 mm
- net Net-(U21A-D): track 14.8 -> 12.4 mm
- net Q_{FF4}: track 30.1 -> 32.4 mm
- net Net-(U14A-D): track 14.8 -> 12.6 mm
- net Net-(U1A-D): track 14.1 -> 12.2 mm
- net V_{Counteroverflow}: track 130.4 -> 129.1 mm
- net Net-(U0A-D): track 14.8 -> 13.6 mm
- net GND: vias 38 -> 40
