File: Capacitijdmeter_ontwerp_counter/Capacitijdmeter_ontwerp_counter.kicad_sch (KiCad schematic)
At the start: 50 parts, among them J1 Screw_Terminal_01x02, J2 Screw_Terminal_01x02, J3 Screw_Terminal_01x02, SW1 SW_MEC_5G, U0 74HC74, U1 74HC74, U10 4511, U12 7408, U14 74HC74, U15 74HC74, U16 4511, U2 7408, U20 74HC74, U21 74HC74, U22 4511, U3 4511, U7 74HC02, U8 74HC74, U9 74HC74

Commit message: "goeiemorgen Koen, ga opnieuw alle traces doen"
Parts:
- removed C1: 1u, Capacitor_THT:C_Radial_D6.3mm_H5.0mm_P2.50mm, symbol Device:C_Polarized
- removed R1: 10k, Resistor_THT:R_Axial_DIN0207_L6.3mm_D2.5mm_P10.16mm_Horizontal, symbol Device:R
- removed SW1: SW_MEC_5G, symbol Switch:SW_MEC_5G
- added J4: Screw_Terminal_01x02, TerminalBlock:TerminalBlock_MaiXu_MX126-5.0-02P_1x02_P5.00mm, symbol Connector:Screw_Terminal_01x02
- added TP8, TP9: TestPoint, Connector_PinHeader_1.00mm:PinHeader_1x01_P1.00mm_Vertical, symbol Connector:TestPoint
Connections:
- net GND: now also J4.2 (Pin_2)
- net Q_{FF10}: now also U16.2 (DC); no longer U10.2 (DC)
- net Q_{FF11}: now also U16.6 (DD); no longer U10.6 (DD)
- net Q_{FF3}: now also U21.12 (D); no longer U21.9 (Q)
- net Q_{FF4}: now also U10.7 (DA); no longer U16.7 (DA)
- net Q_{FF5}: now also U10.1 (DB); no longer U16.1 (DB)
- net Q_{FF6}: now also U10.2 (DC); no longer U16.2 (DC)
- net Q_{FF7}: now also U10.6 (DD); no longer U16.6 (DD)
- net Q_{FF8}: now also U16.7 (DA); no longer U10.7 (DA)
- net Q_{FF9}: now also U16.1 (DB); no longer U10.1 (DB)
- net V_{CounterMR}: now also J4.1 (Pin_1)
- net at U21.2 (D), U21.6 (~{Q}): no longer U21.11 (C)
- net at U21.8 (~{Q}): no longer U21.12 (D)
- net at U20.11 (C), U20.2 (D), U20.6 (~{Q}): now also TP8.1
- net at U1.12 (D), U1.8 (~{Q}): now also TP9.1

Commit message: "PCB Fucking ontwerp"
Parts:
- removed C2, C3: 1u, Capacitor_THT:C_Radial_D6.3mm_H5.0mm_P2.50mm, symbol Device:C_Polarized
- removed C23: 100nF, Capacitor_SMD:C_1206_3216Metric_Pad1.33x1.80mm_HandSolder, symbol Device:C
- removed J1, J2, J3, J4: Screw_Terminal_01x02, TerminalBlock:TerminalBlock_MaiXu_MX126-5.0-02P_1x02_P5.00mm, symbol Connector:Screw_Terminal_01x02
- removed TP4: TestPoint, Connector_PinHeader_1.00mm:PinHeader_1x01_P1.00mm_Vertical, symbol Connector:TestPoint
- added J3: DE9_Pins_MountingHoles, Connector_Dsub:DSUB-9_Pins_Horizontal_P2.77x2.84mm_EdgePinOffset7.70mm_Housed_MountingHolesOffset9.12mm, symbol Connector:DE9_Pins_MountingHoles
- added R1, R2, R3, R4: 10k, Resistor_THT:R_Axial_DIN0207_L6.3mm_D2.5mm_P10.16mm_Horizontal, symbol Device:R
- added TP10, TP11: TestPoint, Connector_PinHeader_1.00mm:PinHeader_1x01_P1.00mm_Vertical, symbol Connector:TestPoint
- U11, U17, U23, U26: footprint Display_7Segment:D1X8K -> footprints:SC56-11EWA_KNB
Connections:
- net +5V: now also J3.6, J3.9, TP11.1
- net GND: now also J3.5, J3.7, J3.SH (PAD), R1.2, R2.2, R3.2, R4.2; no longer U11.3 (CC), U11.8 (CC), U17.3 (CC), U17.8 (CC), U23.3 (CC), U23.5 (DP), U23.8 (CC), U26.3 (CC), U26.8 (CC)
- net Q_{FF3}: now also U21.9 (Q); no longer U21.12 (D)
- net V_{CounterMR}: now also TP7.1, J3.3; no longer TP5.1
- net V_{oneshot}: now also TP5.1, J3.4; no longer TP7.1
- net V_{oscillator}: now also J3.8
- net at U21.11 (C): now also U21.2 (D), U21.6 (~{Q})
- net at U21.8 (~{Q}): now also U21.12 (D)
- net V_{counteroverflow} renamed V_{Counteroverflow}
- net V_{Counteroverflow}: now also J3.2, TP10.1
- new net: R4.1, U26.3 (CC), U26.8 (CC)
- new net: R2.1, U23.3 (CC), U23.8 (CC)
- new net: R1.1, U11.3 (CC), U11.8 (CC)
- new net: R3.1, U17.3 (CC), U17.8 (CC)

Commit message: "alles behalve de ding geroute"
Parts:
- C11, C12, C13, C17, C21: KiLib_Generator (none) -> SMD_2terminal_chip_molded
- J3: KiLib_Generator (none) -> connector/D_sub
- R1, R3, R4: footprint Resistor_THT:R_Axial_DIN0207_L6.3mm_D2.5mm_P10.16mm_Horizontal -> Resistor_SMD:R_1206_3216Metric_Pad1.30x1.75mm_HandSolder
- R2: footprint Resistor_THT:R_Axial_DIN0207_L6.3mm_D2.5mm_P10.16mm_Horizontal -> Resistor_SMD:R_1206_3216Metric_Pad1.30x1.75mm_HandSolder; KiLib_Generator (none) -> SMD_2terminal_chip_molded
- TP10, TP11, TP5, TP6, TP7, TP8, TP9: KiLib_Generator (none) -> connector/pin_header_socket
- U12, U2, U20, U21, U22, U7: KiLib_Generator (none) -> package/gullwing

Commit message: "flipping hell, Koen, hier asjeblieft"
Changed lines of the file:
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@@
 	)
 	(junction
-		(at 224.79 228.6)
-		(diameter 0)
-		(color 0 0 0 0)
-	)
-	(junction
 		(at 261.62 118.11)
 		(diameter 0)
@@
 	(wire
 		(pts
-			(xy 218.44 228.6) (xy 224.79 228.6)
-		)
-		(stroke
-			(width 0)
-			(type default)
-		)
-	)
-	(wire
-		(pts
 			(xy 236.22 168.91) (xy 248.92 168.91)
 		)
@@
 	(wire
 		(pts
-			(xy 224.79 227.33) (xy 224.79 228.6)
-		)
-		(stroke
-			(width 0)
-			(type default)
-		)
-	)
-	(wire
-		(pts
 			(xy 104.14 184.15) (xy 100.33 184.15)
 		)
@@
 	(wire
 		(pts
-			(xy 224.79 228.6) (xy 224.79 247.65)
+			(xy 224.79 227.33) (xy 224.79 247.65)
 		)
 		(stroke

Commit message: s
Parts:
- removed TP10: TestPoint, Connector_PinHeader_1.00mm:PinHeader_1x01_P1.00mm_Vertical, symbol Connector:TestPoint
- removed U12: 7408, Package_SO:SOIC-14_3.9x8.7mm_P1.27mm, symbol 74xx_IEEE:7408
- added C14: 100nF, Capacitor_SMD:C_1206_3216Metric_Pad1.33x1.80mm_HandSolder, symbol Device:C
- added U4: 7402, Package_SO:SOIC-14_3.9x8.7mm_P1.27mm, symbol 74xx:7402
- added U5: 7411, Package_SO:SOIC-14_3.9x8.7mm_P1.27mm, symbol 74xx_IEEE:7411
Connections:
- net +5V: now also C14.2, U4.14 (VCC), U5.14 (VCC), U5.14 (VCC), U5.14 (VCC)
- net GND: now also J3.2, C14.1, U4.2, U4.3, U4.5, U4.6, U4.7 (GND), U5.10, U5.11, U5.3, U5.4, U5.5, U5.7 (GND), U5.7 (GND), U5.7 (GND), U5.9
- net V_{CounterMR}: now also U4.12
- net V_{Counteroverflow}: now also U4.8; no longer J3.2
- net V_{input_counter}: now also U5.12
- net V_{oneshot}: now also U5.2
- net V_{oscillator}: now also U5.1
- net reset_0: no longer names the net of U20.1 (~{R}), U20.13 (~{R}), U21.1 (~{R}), U21.13 (~{R}), U7.13
- net reset_1: no longer names the net of U7.4, U8.1 (~{R}), U8.13 (~{R}), U9.1 (~{R}), U9.13 (~{R})
- net reset_2: no longer names the net of U14.1 (~{R}), U14.13 (~{R}), U15.1 (~{R}), U15.13 (~{R}), U7.10
- new net: U4.13, U4.9
- new net V_{Counterstop}: U4.10, U4.11, U5.13

Commit message: dih
Other:
- moved on the sheet: C10, C11, C12, C13, C14, C16, C17, C18, C19, C20, C21, C5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

Commit message: "NIEUWE VERSIE ERIN GEKNIKKERD MET EEN PCB DAT BIJNA KLAAR IS"
Connections:
- net GND: now also J3.1
Other:
- moved on the sheet: C10, C11, C12, C13, C14, C16, C17, C18, C19, C20, C21, C5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

Commit message: "ALL COMMIT"
Parts:
- R1, R2, R3, R4: value 10k -> 500
Connections:
- net GND: now also U23.5 (DP)
Changed lines of the file:
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@@
 	(wire
 		(pts
-			(xy 283.21 36.83) (xy 283.21 49.53)
-		)
-		(stroke
-			(width 0)
-			(type default)
-		)
-	)
-	(wire
-		(pts
 			(xy -25.4 184.15) (xy -25.4 191.77)
 		)
@@
 	(wire
 		(pts
+			(xy 283.21 36.83) (xy 283.21 49.53)
+		)
+		(stroke
+			(width 0)
+			(type default)
+		)
+	)
+	(wire
+		(pts
 			(xy 389.89 236.22) (xy 398.78 236.22)
 		)
@@
 			)
 		)
-		(property "Value" "10k"
+		(property "Value" "500"
 			(at 285.75 62.2299 0)
 			(show_name no)
@@
 	)
 	(symbol
+		(lib_id "power:GND")
+		(at 290.83 41.91 270)
+		(unit 1)
+		(body_style 1)
+		(exclude_from_sim no)
+		(in_bom yes)
+		(on_board yes)
+		(in_pos_files yes)
+		(dnp no)
+		(fields_autoplaced yes)
+		(property "Reference" "#PWR087"
+			(at 284.48 41.91 0)
+			(hide yes)
+			(show_name no)
+			(do_not_autoplace no)
+			(effects
+				(font
+					(size 1.27 1.27)
+				)
+			)
+		)
+		(property "Value" "GND"
+			(at 287.02 41.9099 90)
+			(show_name no)
+			(do_not_autoplace no)
+			(effects
+				(font
+					(size 1.27 1.27)
+				)
+				(justify right)
+			)
+		)
+		(property "Footprint" ""
+			(at 290.83 41.91 0)
+			(hide yes)
+			(show_name no)
+			(do_not_autoplace no)
+			(effects
+				(font
+					(size 1.27 1.27)
+				)
+			)
+		)
+		(property "Datasheet" ""
+			(at 290.83 41.91 0)
+			(hide yes)
+			(show_name no)
+			(do_not_autoplace no)
+			(effects
+				(font
+					(size 1.27 1.27)
+				)
+			)
+		)
+		(property "Description" "Power symbol creates a global label with name \"GND\" , ground"
+			(at 290.83 41.91 0)
+			(hide yes)
+			(show_name no)
+			(do_not_autoplace no)
+			(effects
+				(font
+					(size 1.27 1.27)
+				)
+			)
+		)
+		(pin "1"
+		)
+		(instances
+			(project "Capacitijdmeter_ontwerp_counter"
+				(path "/6aee43a7-1066-4186-960d-016fada1ad3c"
+					(reference "#PWR087")
+					(unit 1)
+				)
+			)
+		)
+	)
+	(symbol
 		(lib_id "power:+5V")
 		(at 375.92 92.71 0)
@@
 			)
 		)
-		(property "Value" "10k"
+		(property "Value" "500"
 			(at 293.37 240.0299 0)
 			(show_name no)
@@
 			)
 		)
-		(property "Value" "10k"
+		(property "Value" "500"
 			(at 281.94 190.4999 0)
 			(show_name no)
@@
 			)
 		)
-		(property "Value" "10k"
+		(property "Value" "500"
 			(at 284.48 119.3799 0)
 			(show_name no)
