File: Capacitijdmeter_ontwerp_counter_AUTOTRACING/Capacitijdmeter_ontwerp_counter.kicad_pcb (KiCad board)
At the start: 2 copper layers, 123.6 x 70.8 mm, 50 parts, among them J3 DE9_Pins_MountingHoles, U0 74HC74, U1 74HC74, U10 4511, U14 74HC74, U15 74HC74, U16 4511, U2 7408, U20 74HC74, U21 74HC74, U22 4511, U3 4511, U4 7402, U5 7411, U7 74HC02, U8 74HC74, U9 74HC74

Commit message: "DE AFGEMAAKTE PCB VAN DE COUNTER"
Parts:
- moved TP11 5.08 mm to (137.2, 61.0)
Routing:
- net V_{b1}: track 27.0 -> 30.3 mm
- net V_{b0}: track 27.0 -> 30.3 mm
- net +5V: track 867.2 -> 870.4 mm
- net V_{b2}: track 27.0 -> 30.2 mm
- net V_{a0}: track 32.1 -> 35.3 mm
- net V_{a1}: track 32.1 -> 35.1 mm
- net V_{a2}: track 32.1 -> 35.0 mm
- net V_{b3}: track 27.0 -> 29.4 mm
- net V_{a3}: track 32.1 -> 34.2 mm
- net reset_3: track 96.4 -> 97.2 mm
- net V_{f0}: track 40.5 -> 41.0 mm
- net V_{g0}: track 32.7 -> 33.2 mm
- net GND: vias 33 -> 38
Other:
- board size 123.6 x 70.8 mm -> 118.5 x 80.8 mm
